File: USB4125-GF-A_Breakout-Board.kicad_sch (KiCad schematic)
At the start: 6 parts, among them J1 Conn_01x04_Male, J2 Conn_01x03_Male, J3 USB4125-GF-A

Commit message: Mod: Finished project, updated schematic, added pcb and panel and exported data
Parts:
- J1: footprint (none) -> Connector_PinHeader_2.54mm:PinHeader_1x04_P2.54mm_Vertical
- J3: footprint ZigbeeZwaveEthernetadapter:GCT_USB4125-GF-A -> connectors:GCT_USB4125-GF-A
- JP1: footprint (none) -> Jumper:SolderJumper-2_P1.3mm_Open_RoundedPad1.0x1.5mm
Connections:
- net CC1: now reaches J1.3 (Pin_3), J3.A5 (CC1), R1.1
- net SHIELD: now reaches J2.3 (Pin_3), J3.S1 (SHIELD), JP1.2 (B)
- net VBUS: now reaches J1.1 (Pin_1), J1.2 (Pin_2), J3.A9 (VBUS), J3.B9 (VBUS)
- net CC2: now reaches J1.4 (Pin_4), J3.B5 (CC2), R2.1
Changed lines of the file:
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@@
     (stroke (width 0) (type default) (color 0 0 0 0))
+  )
+  (label "CC1" (at 152.4 86.36 0)
+    (effects (font (size 1.27 1.27)) (justify left bottom))
+  )
+  (label "SHIELD" (at 152.4 116.84 0)
+    (effects (font (size 1.27 1.27)) (justify left bottom))
+  )
+  (label "GND" (at 152.4 111.76 0)
+    (effects (font (size 1.27 1.27)) (justify left bottom))
+  )
+  (label "CC2" (at 152.4 88.9 0)
+    (effects (font (size 1.27 1.27)) (justify left bottom))
+  )
+  (label "VBUS" (at 152.4 78.74 0)
+    (effects (font (size 1.27 1.27)) (justify left bottom))
   )
   (symbol (lib_id "Device:R") (at 139.7 95.25 0) (unit 1)
@@
     (property "Reference" "JP1" (id 0) (at 152.4 120.65 0))
     (property "Value" "SolderJumper_2_Open" (id 1) (at 152.4 123.19 0))
-    (property "Footprint" "" (id 2) (at 152.4 127 0)
+    (property "Footprint" "Jumper:SolderJumper-2_P1.3mm_Open_RoundedPad1.0x1.5mm" (id 2) (at 152.4 127 0)
       (effects (font (size 1.27 1.27)) hide)
     )
@@
       (effects (font (size 1.27 1.27)) (justify left))
     )
-    (property "Footprint" "ZigbeeZwaveEthernetadapter:GCT_USB4125-GF-A" (id 2) (at 177.8 90.17 0)
+    (property "Footprint" "connectors:GCT_USB4125-GF-A" (id 2) (at 177.8 90.17 0)
       (effects (font (size 1.27 1.27)) (justify bottom) hide)
     )
@@
       (effects (font (size 1.27 1.27)) (justify right))
     )
-    (property "Footprint" "" (id 2) (at 114.3 81.28 0)
+    (property "Footprint" "Connector_PinHeader_2.54mm:PinHeader_1x04_P2.54mm_Vertical" (id 2) (at 114.3 81.28 0)
       (effects (font (size 1.27 1.27)) hide)
     )
@@
     )
     (path "/a4d0cdeb-aee1-4a62-b293-804f36ae4062"
-      (reference "J3") (unit 1) (value "USB4125-GF-A") (footprint "ZigbeeZwaveEthernetadapter:GCT_USB4125-GF-A")
+      (reference "J3") (unit 1) (value "USB4125-GF-A") (footprint "connectors:GCT_USB4125-GF-A")
     )
     (path "/70b339c3-6aac-4c1c-8fba-7087bf98781d"
