File: USB4125-GF-A_Breakout-Board.kicad_pcb (KiCad board)
At the start: 2 copper layers, 20.3 x 15.2 mm, 7 parts, among them J1 Conn_01x04_Male, J2 Conn_01x03_Male, J3 USB4125-GF-A

Commit message: Mod: Updated the project name and revision to be on the copper layer now
Routing:
- net GND: vias 6 -> 5
Other:
- board text added: "${TITLE} Rev: ${REVISION}"
- board text removed: "Prj: ${TITLE} Rev: ${REVISION}"
Changed lines of the file:
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@@
   (title_block
     (title "USB4125-GF-A Breakout Board")
-    (date "2023-03-06")
-    (rev "A")
+    (date "2023-03-07")
+    (rev "B")
     (company "ElektroNik Zoller")
     (comment 1 "Nikolai Zoller")
@@
   )
   (gr_rect (start 124.46 87.63) (end 144.78 102.87) (layer "Edge.Cuts") (width 0.1) (fill none))
-  (gr_text "Prj: ${TITLE}\nRev: ${REVISION}" (at 134.62 101.346) (layer "B.Mask")
-    (effects (font (size 0.4 0.4) (thickness 0.1)) (justify mirror))
+  (gr_text "${TITLE}\nRev: ${REVISION}" (at 144.145 101.346) (layer "B.Cu")
+    (effects (font (size 0.6 0.6) (thickness 0.15)) (justify left mirror))
   )
   (via (at 140.462 94.234) (size 0.8) (drill 0.4) (layers "F.Cu" "B.Cu") (free) (net 1))
-  (via (at 142.24 100.965) (size 0.8) (drill 0.4) (layers "F.Cu" "B.Cu") (free) (net 1))
-  (via (at 129.54 99.695) (size 0.8) (drill 0.4) (layers "F.Cu" "B.Cu") (free) (net 1))
+  (via (at 129.032 99.06) (size 0.8) (drill 0.4) (layers "F.Cu" "B.Cu") (free) (net 1))
   (via (at 139.192 97.028) (size 0.8) (drill 0.4) (layers "F.Cu" "B.Cu") (free) (net 1))
   (via (at 127 89.535) (size 0.8) (drill 0.4) (layers "F.Cu" "B.Cu") (free) (net 1))
